Commit message: change joint type of some parts and the position of omnicam

File: urdf_model/urdf/ex1.urdf (robot description, URDF)
Before this commit: robot EX1, 34 links, 33 joints
Joints:
- joint Left_leg_joint: type continuous -> fixed
- joint Right_leg_joint: type continuous -> fixed
- joint camera_case_joint: type continuous -> fixed
- joint omnicam_base_joint: origin xyz=0.0 0 0.25 -> xyz=0 0 0.2225
- joint omnicam_joint: origin xyz=0.0 0 0 rpy=0 1.570795 0 -> xyz=0 0 -0.2 rpy=0 1.570795 0

Commit message: Update EX1 urdf
Changed the joint type of some parts, and the way of defining the gazebo color

File: urdf_model/urdf/ex1.urdf (robot description, URDF)
Before this commit: robot EX1, 34 links, 33 joints
Joints:
- joint Lfsteering_joint: type continuous -> fixed
- joint Rfsteering_joint: type continuous -> fixed
